Commit message: Fix

File: urdf/wamv_base.urdf.xacro (robot description, xacro)
@@ -85,5 +85,5 @@
     <visual>
       <geometry>
-        <mesh filename="package://rowbot_description/mesh/WAM-V-Base.dae" s/>
+        <mesh filename="package://rowbot_description/mesh/WAM-V-Base.dae"/>
       </geometry>
     </visual>
