Commit message: Mesh update

File: urdf/engine.xacro (robot description, xacro)
@@ -6,5 +6,5 @@
       <visual>
         <geometry>
-          <mesh filename="package://wamv_description/mesh/engine.dae"/>
+          <mesh filename="package://rowbot_description/mesh/engine.dae"/>
         </geometry>
       </visual>
@@ -29,5 +29,5 @@
       <visual>
         <geometry>
-          <mesh filename="package://wamv_description/mesh/propeller.dae"/>
+          <mesh filename="package://rowbot_description/mesh/propeller.dae"/>
         </geometry>
       </visual>

File: urdf/wamv_base.urdf.xacro (robot description, xacro)
@@ -85,5 +85,5 @@
     <visual>
       <geometry>
-        <mesh filename="package://wamv_description/mesh/WAM-V-Base.dae"/>
+        <mesh filename="package://rowbot_description/mesh/WAM-V-Base.dae"/>
       </geometry>
     </visual>

Commit message: Scale

File: urdf/engine.xacro (robot description, xacro)
@@ -6,5 +6,5 @@
       <visual>
         <geometry>
-          <mesh filename="package://rowbot_description/mesh/engine.dae"/>
+          <mesh filename="package://rowbot_description/mesh/engine.dae" scale="0.001 0.001 0.001"/>
         </geometry>
       </visual>
@@ -29,5 +29,5 @@
       <visual>
         <geometry>
-          <mesh filename="package://rowbot_description/mesh/propeller.dae"/>
+          <mesh filename="package://rowbot_description/mesh/propeller.dae" scale="0.001 0.001 0.001"/>
         </geometry>
       </visual>
@@ -53,6 +53,6 @@
       <child link="${prefix}_propeller_link"/>
       <origin rpy="0 0 0" xyz="-0.278156 0 -0.509371"/>
-      <limit effort="100" velocity="100" />
-      <dynamics friction="0.05" damping="0.05" />
+      <!--limit effort="100" velocity="100" />
+      <dynamics friction="0.05" damping="0.05" /-->
     </joint>
   </xacro:macro>

File: urdf/wamv_base.urdf.xacro (robot description, xacro)
@@ -85,5 +85,5 @@
     <visual>
       <geometry>
-        <mesh filename="package://rowbot_description/mesh/WAM-V-Base.dae"/>
+        <mesh filename="package://rowbot_description/mesh/WAM-V-Base.dae" scale="0.001 0.001 0.001"/>
       </geometry>
     </visual>

Commit message: Scale 2

File: urdf/engine.xacro (robot description, xacro)
@@ -6,5 +6,5 @@
       <visual>
         <geometry>
-          <mesh filename="package://rowbot_description/mesh/engine.dae" scale="0.001 0.001 0.001"/>
+          <mesh filename="package://rowbot_description/mesh/engine.dae" />
         </geometry>
       </visual>
@@ -29,5 +29,5 @@
       <visual>
         <geometry>
-          <mesh filename="package://rowbot_description/mesh/propeller.dae" scale="0.001 0.001 0.001"/>
+          <mesh filename="package://rowbot_description/mesh/propeller.dae" />
         </geometry>
       </visual>

File: urdf/wamv_base.urdf.xacro (robot description, xacro)
@@ -85,5 +85,5 @@
     <visual>
       <geometry>
-        <mesh filename="package://rowbot_description/mesh/WAM-V-Base.dae" scale="0.001 0.001 0.001"/>
+        <mesh filename="package://rowbot_description/mesh/WAM-V-Base.dae" s/>
       </geometry>
     </visual>

Commit message: Scale3

File: urdf/engine.xacro (robot description, xacro)
@@ -6,5 +6,5 @@
       <visual>
         <geometry>
-          <mesh filename="package://rowbot_description/mesh/engine.dae" />
+          <mesh filename="package://rowbot_description/mesh/engine.dae" scale="0.01 0.01 0.01"/>
         </geometry>
       </visual>
@@ -29,5 +29,5 @@
       <visual>
         <geometry>
-          <mesh filename="package://rowbot_description/mesh/propeller.dae" />
+          <mesh filename="package://rowbot_description/mesh/propeller.dae" scale="0.01 0.01 0.01"/>
         </geometry>
       </visual>

File: urdf/wamv_base.urdf.xacro (robot description, xacro)
@@ -85,5 +85,5 @@
     <visual>
       <geometry>
-        <mesh filename="package://rowbot_description/mesh/WAM-V-Base.dae"/>
+        <mesh filename="package://rowbot_description/mesh/WAM-V-Base.dae" scale="0.01 0.01 0.01"/>
       </geometry>
     </visual>

Commit message: Fixed propellor

File: urdf/engine.xacro (robot description, xacro)
@@ -48,5 +48,5 @@
       <child link="${prefix}_engine_link"/>
     </joint>
-    <joint name="${prefix}_engine_propeller_joint" type="continuous">
+    <joint name="${prefix}_engine_propeller_joint" type="fixed">
       <axis rpy="0 0 0" xyz="1 0 0"/>
       <parent link="${prefix}_engine_link"/>

Commit message: FIxed

File: urdf/engine.xacro (robot description, xacro)
@@ -49,5 +49,4 @@
     </joint>
     <joint name="${prefix}_engine_propeller_joint" type="fixed">
-      <axis rpy="0 0 0" xyz="1 0 0"/>
       <parent link="${prefix}_engine_link"/>
       <child link="${prefix}_propeller_link"/>
