Commit message: changed some configuration

File: urdf/sensors/wamv_3d_lidar.xacro (robot description, xacro)
@@ -13,5 +13,5 @@
     noise_stddev: Standard deviation of gaussian noise applied to output pointcloud
   -->
-  <xacro:macro name="wamv_3d_lidar" params="name x:=0.7 y:=0 z:=1.45 R:=0 P:=0 Y:=0
+  <xacro:macro name="wamv_3d_lidar" params="name x:=0.75 y:=0 z:=1.45 R:=0 P:=0 Y:=-0.08
                                             update_rate:=10 vertical_lasers:=16 samples:=1800 resolution:=0.5
                                             min_angle:=${-pi} max_angle:=${pi}
